File: Hardware/EC60_1.brd (EAGLE design)
At the start: 66 x 66 mm, 4 parts

Commit message: Some Changes
Parts:
- SK1: device jt-con-micromatch:AMP-215079-10 -> microMatch:AMP-215079-10
Changed lines of the file:
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@@
 <?xml version="1.0" encoding="utf-8"?>
 <!DOCTYPE eagle SYSTEM "eagle.dtd">
-<eagle version="7.5.0">
+<eagle version="8.6.0">
 <drawing>
 <settings>
 <setting alwaysvectorfont="yes"/>
+<setting keepoldvectorfont="yes"/>
 <setting verticaltext="up"/>
 </settings>
@@
 <layer number="2" name="Route2" color="1" fill="3" visible="no" active="no"/>
 <layer number="3" name="Route3" color="4" fill="3" visible="no" active="no"/>
+<layer number="4" name="Route4" color="1" fill="4" visible="no" active="yes"/>
+<layer number="5" name="Route5" color="4" fill="4" visible="no" active="yes"/>
+<layer number="6" name="Route6" color="1" fill="8" visible="no" active="yes"/>
+<layer number="7" name="Route7" color="4" fill="8" visible="no" active="yes"/>
+<layer number="8" name="Route8" color="1" fill="2" visible="no" active="yes"/>
+<layer number="9" name="Route9" color="4" fill="2" visible="no" active="yes"/>
+<layer number="10" name="Route10" color="1" fill="7" visible="no" active="yes"/>
+<layer number="11" name="Route11" color="4" fill="7" visible="no" active="yes"/>
+<layer number="12" name="Route12" color="1" fill="5" visible="no" active="yes"/>
+<layer number="13" name="Route13" color="4" fill="5" visible="no" active="yes"/>
 <layer number="14" name="Route14" color="1" fill="6" visible="no" active="no"/>
 <layer number="15" name="Route15" color="4" fill="6" visible="no" active="no"/>
@@
 &lt;/ul&gt;
 &lt;/p&gt;</description>
+<fusionsync huburn="a.cGVyc29uYWw6dWUyOWRmMDE1" projecturn="a.cGVyc29uYWw6dWUyOWRmMDE1IzIwMTgwMTA0MTEwODc3NDI2" f3durn="urn:adsk.wipprod:dm.lineage:H2HDAAFKQPivREwpPJ56ww" pcbguid="41bf4e22-6b47-41d1-9a15-bb805b3d37d7" lastpulledtime="" lastsyncedchangeguid="9ca032c8-7506-94c8-c300-a7ab2aa5612a"/>
 <plain>
 <wire x1="0" y1="0" x2="66.02" y2="0" width="0" layer="20"/>
@@
 <param name="dpMaxLengthDifference" value="10mm"/>
 <param name="dpGapFactor" value="2.5"/>
-<param name="checkGrid" value="0"/>
 <param name="checkAngle" value="0"/>
 <param name="checkFont" value="1"/>
 <param name="checkRestrict" value="0"/>
+<param name="checkStop" value="0"/>
+<param name="checkValues" value="0"/>
 <param name="useDiameter" value="13"/>
 <param name="maxErrors" value="50"/>
@@
 <element name="JP1" library="pinhead" package="1X03" value="K1" x="45.5113375" y="33.00031875" rot="R270"/>
 <element name="JP2" library="pinhead" package="1X03" value="K2" x="20.445878125" y="33.00031875" rot="R90"/>
-<element name="U$1" library="ALPS-EC60A" package="EC60A" value="EC60A" x="33.000096875" y="33.00021875"/>
-<element name="SK1" library="jt-con-micromatch" package="AMP-215079-10" value="Keys" x="38.8" y="54.9" rot="MR0"/>
+<element name="U$1" library="ALPS-EC60A" library_urn="urn:adsk.eagle:library:1567918" package="EC60A" package3d_urn="urn:adsk.eagle:package:1567921/2" value="EC60A" x="33.000096875" y="33.00021875"/>
+<element name="SK1" library="microMatch" library_urn="urn:adsk.eagle:library:353375" package="AMP-215079-10" package3d_urn="urn:adsk.eagle:package:353401/2" value="Keys" x="38.8" y="54.9" rot="MR0"/>
 </elements>
 <signals>
@@
 </board>
 </drawing>
+<compatibility>
+<note version="8.2" severity="warning">
+Since Version 8.2, EAGLE supports online libraries. The ids
+of those online libraries will not be understood (or retained)
+with this version.
+</note>
+<note version="8.3" severity="warning">
+Since Version 8.3, EAGLE supports Fusion synchronisation.
+This feature will not be available in this version and saving
+the document will break the link to the Fusion PCB feature.
+</note>
+<note version="8.3" severity="warning">
+Since Version 8.3, EAGLE supports URNs for individual library
+assets (packages, symbols, and devices). The URNs of those assets
+will not be understood (or retained) with this version.
+</note>
+<note version="8.3" severity="warning">
+Since Version 8.3, EAGLE supports the association of 3D packages
+with devices in libraries, schematics, and board files. Those 3D
+packages will not be understood (or retained) with this version.
+</note>
+</compatibility>
 </eagle>
