File: Hardware/EC60_1.sch (EAGLE design)
At the start: 4 parts

Commit message: Some Changes
Parts:
- SK1: device jt-con-micromatch:MMATCH-10-PTH -> microMatch:MMATCH-10-PTH
Changed lines of the file:
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@@
 <?xml version="1.0" encoding="utf-8"?>
 <!DOCTYPE eagle SYSTEM "eagle.dtd">
-<eagle version="7.5.0">
+<eagle version="8.6.0">
 <drawing>
 <settings>
 <setting alwaysvectorfont="yes"/>
+<setting keepoldvectorfont="yes"/>
 <setting verticaltext="up"/>
 </settings>
@@
 <layer number="2" name="Route2" color="1" fill="3" visible="no" active="no"/>
 <layer number="3" name="Route3" color="4" fill="3" visible="no" active="no"/>
+<layer number="4" name="Route4" color="1" fill="4" visible="no" active="no"/>
+<layer number="5" name="Route5" color="4" fill="4" visible="no" active="no"/>
+<layer number="6" name="Route6" color="1" fill="8" visible="no" active="no"/>
+<layer number="7" name="Route7" color="4" fill="8" visible="no" active="no"/>
+<layer number="8" name="Route8" color="1" fill="2" visible="no" active="no"/>
+<layer number="9" name="Route9" color="4" fill="2" visible="no" active="no"/>
+<layer number="10" name="Route10" color="1" fill="7" visible="no" active="no"/>
+<layer number="11" name="Route11" color="4" fill="7" visible="no" active="no"/>
+<layer number="12" name="Route12" color="1" fill="5" visible="no" active="no"/>
+<layer number="13" name="Route13" color="4" fill="5" visible="no" active="no"/>
 <layer number="14" name="Route14" color="1" fill="6" visible="no" active="no"/>
 <layer number="15" name="Route15" color="4" fill="6" visible="no" active="no"/>
@@
 </classes>
 <parts>
-<part name="U$1" library="ALPS-EC60A" deviceset="EC60A" device=""/>
+<part name="U$1" library="ALPS-EC60A" library_urn="urn:adsk.eagle:library:1567918" deviceset="EC60A" device="" package3d_urn="urn:adsk.eagle:package:1567921/2"/>
 <part name="FRAME1" library="frames" deviceset="A4L-LOC" device="" value="Encoder"/>
 <part name="JP1" library="pinhead" deviceset="PINHD-1X3" device="" value="K1"/>
 <part name="JP2" library="pinhead" deviceset="PINHD-1X3" device="" value="K2"/>
-<part name="SK1" library="jt-con-micromatch" deviceset="MMATCH-10-*" device="PTH" value="Keys"/>
+<part name="SK1" library="microMatch" library_urn="urn:adsk.eagle:library:353375" deviceset="MMATCH-10-*" device="PTH" package3d_urn="urn:adsk.eagle:package:353401/2" value="Keys"/>
 </parts>
 <sheets>
@@
 </schematic>
 </drawing>
+<compatibility>
+<note version="8.2" severity="warning">
+Since Version 8.2, EAGLE supports online libraries. The ids
+of those online libraries will not be understood (or retained)
+with this version.
+</note>
+<note version="8.3" severity="warning">
+Since Version 8.3, EAGLE supports URNs for individual library
+assets (packages, symbols, and devices). The URNs of those assets
+will not be understood (or retained) with this version.
+</note>
+<note version="8.3" severity="warning">
+Since Version 8.3, EAGLE supports the association of 3D packages
+with devices in libraries, schematics, and board files. Those 3D
+packages will not be understood (or retained) with this version.
+</note>
+</compatibility>
 </eagle>
