File: Hardware/TFT-Board.brd (EAGLE design)
At the start: 68 x 34 mm, 5 parts, among them Q1 2N3906

Commit message: Some Changes
Parts:
- R1, R2: device resistor:0204/7 -> PartCollection:0204/7
- SK1: device jt-con-micromatch:AMP-215079-10 -> microMatch:AMP-215079-10
Changed lines of the file:
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@@
 <?xml version="1.0" encoding="utf-8"?>
 <!DOCTYPE eagle SYSTEM "eagle.dtd">
-<eagle version="7.5.0">
+<eagle version="8.6.0">
 <drawing>
 <settings>
 <setting alwaysvectorfont="yes"/>
+<setting keepoldvectorfont="yes"/>
 <setting verticaltext="up"/>
 </settings>
@@
 <layer number="2" name="Route2" color="1" fill="3" visible="no" active="no"/>
 <layer number="3" name="Route3" color="4" fill="3" visible="no" active="no"/>
+<layer number="4" name="Route4" color="1" fill="4" visible="no" active="yes"/>
+<layer number="5" name="Route5" color="4" fill="4" visible="no" active="yes"/>
+<layer number="6" name="Route6" color="1" fill="8" visible="no" active="yes"/>
+<layer number="7" name="Route7" color="4" fill="8" visible="no" active="yes"/>
+<layer number="8" name="Route8" color="1" fill="2" visible="no" active="yes"/>
+<layer number="9" name="Route9" color="4" fill="2" visible="no" active="yes"/>
+<layer number="10" name="Route10" color="1" fill="7" visible="no" active="yes"/>
+<layer number="11" name="Route11" color="4" fill="7" visible="no" active="yes"/>
+<layer number="12" name="Route12" color="1" fill="5" visible="no" active="yes"/>
+<layer number="13" name="Route13" color="4" fill="5" visible="no" active="yes"/>
 <layer number="14" name="Route14" color="1" fill="6" visible="no" active="no"/>
 <layer number="15" name="Route15" color="4" fill="6" visible="no" active="no"/>
@@
 <layer number="54" name="bGND_GNDA" color="1" fill="9" visible="no" active="no"/>
 <layer number="56" name="wert" color="7" fill="1" visible="yes" active="yes"/>
+<layer number="88" name="SimResults" color="9" fill="1" visible="no" active="no"/>
+<layer number="89" name="SimProbes" color="9" fill="1" visible="no" active="no"/>
 <layer number="90" name="Modules" color="5" fill="1" visible="no" active="no"/>
 <layer number="91" name="Nets" color="2" fill="1" visible="no" active="no"/>
@@
 </layers>
 <board>
+<fusionsync huburn="a.cGVyc29uYWw6dWUyOWRmMDE1" projecturn="a.cGVyc29uYWw6dWUyOWRmMDE1IzIwMTgwMTA0MTEwODc3NDI2" f3durn="urn:adsk.wipprod:dm.lineage:mPl-fwXOQoGFacbh2hTQxw" pcbguid="d9d32e1f-de72-4a1f-bf64-b99d9e673c90" lastpulledtime="" lastsyncedchangeguid="6bcebb4d-2515-3f5e-5459-ed9e9f4f1cf5"/>
 <plain>
 <wire x1="5" y1="24.46" x2="5" y2="18.54" width="0" layer="20"/>
@@
 <param name="dpMaxLengthDifference" value="10mm"/>
 <param name="dpGapFactor" value="2.5"/>
-<param name="checkGrid" value="0"/>
 <param name="checkAngle" value="0"/>
 <param name="checkFont" value="1"/>
 <param name="checkRestrict" value="0"/>
+<param name="checkStop" value="0"/>
+<param name="checkValues" value="0"/>
 <param name="useDiameter" value="13"/>
 <param name="maxErrors" value="50"/>
@@
 <elements>
 <element name="Q1" library="transistor-pnp" package="TO92" value="2N3906" x="53.34" y="5.81" rot="R90"/>
-<element name="R1" library="resistor" package="0204/7" value="100" x="47.02" y="10.08"/>
-<element name="R2" library="resistor" package="0204/7" value="10k" x="43.72" y="4.99"/>
-<element name="U$1" library="2.2&quot;tft" package="2.2_TFT_LCD_LEDSEE" value="2.2_TFT_LCDNEW" x="33.59" y="20.12" rot="MR0"/>
-<element name="SK1" library="jt-con-micromatch" package="AMP-215079-10" value="SPI" x="38.5" y="11" rot="R180"/>
+<element name="R1" library="PartCollection" library_urn="urn:adsk.eagle:library:1606324" package="0204/7" package3d_urn="urn:adsk.eagle:package:1606650/1" value="100" x="47.02" y="10.08"/>
+<element name="R2" library="PartCollection" library_urn="urn:adsk.eagle:library:1606324" package="0204/7" package3d_urn="urn:adsk.eagle:package:1606650/1" value="10k" x="43.72" y="4.99"/>
+<element name="U$1" library="2.2&quot;tft" library_urn="urn:adsk.eagle:library:1567911" package="2.2_TFT_LCD_LEDSEE" package3d_urn="urn:adsk.eagle:package:1567916/2" value="2.2_TFT_LCDNEW" x="33.59" y="20.12" rot="MR0"/>
+<element name="SK1" library="microMatch" library_urn="urn:adsk.eagle:library:353375" package="AMP-215079-10" package3d_urn="urn:adsk.eagle:package:353401/2" value="SPI" x="38.5" y="11" rot="R180"/>
 </elements>
 <signals>
@@
 </board>
 </drawing>
+<compatibility>
+<note version="8.2" severity="warning">
+Since Version 8.2, EAGLE supports online libraries. The ids
+of those online libraries will not be understood (or retained)
+with this version.
+</note>
+<note version="8.3" severity="warning">
+Since Version 8.3, EAGLE supports Fusion synchronisation.
+This feature will not be available in this version and saving
+the document will break the link to the Fusion PCB feature.
+</note>
+<note version="8.3" severity="warning">
+Since Version 8.3, EAGLE supports URNs for individual library
+assets (packages, symbols, and devices). The URNs of those assets
+will not be understood (or retained) with this version.
+</note>
+<note version="8.3" severity="warning">
+Since Version 8.3, EAGLE supports the association of 3D packages
+with devices in libraries, schematics, and board files. Those 3D
+packages will not be understood (or retained) with this version.
+</note>
+</compatibility>
 </eagle>
